File: Qwiic - MMC/SparkFun_9DoF_ISM330DLC-MMC5983MA.sch (EAGLE design)
At the start: 33 parts, among them J1 QWIIC_RIGHT_ANGLE, J2 QWIIC_RIGHT_ANGLE, U1 ISM330DLC, U2 MMC5983MA_QFN16

Commit message: Updates text in schematic referencing old part
Other:
- note added: "ISM330DLC should default to MODE2 (Sensor Hub Mode) to receive MMC5938MA sensor data."
- note removed: "ISM330DHCX should default to MODE2 (Sensor Hub Mode) to receive MMC5938MA sensor data."
Changed lines of the file:
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@@
 <text x="216.916" y="103.632" size="1.778" layer="97" font="vector" align="top-left">Cut traces to remove I2C
 pull-up resistors.</text>
-<text x="55.88" y="190.5" size="1.778" layer="97" font="vector" align="top-left">ISM330DHCX should default to
+<text x="55.88" y="190.5" size="1.778" layer="97" font="vector" align="top-left">ISM330DLC should default to
 MODE2 (Sensor Hub Mode) to receive
 MMC5938MA sensor data.
