File: Qwiic Updated/SparkFun_9DoF_ISM330DHCX-MMC5983MA.sch (EAGLE design)
At the start: 33 parts, among them J1 QWIIC_RIGHT_ANGLE, J2 QWIIC_RIGHT_ANGLE, U1 ISM330DHCX, U2 MMC5983MA_QFN16

Commit message: Adds text to schematic, adds jumpers to SDX and SCX
Parts:
- added SCX, SDX: JUMPER-SMT_2_NC_TRACE_SILK, SparkFun-Jumpers:JUMPER-SMT_2_NC_TRACE_SILK
Connections:
- net GND: now also SCX.1, SDX.1
- net SCX: now also SCX.2
- net SDX: now also SDX.2
Other:
- note added: "Accelerometer Address Selection and Sensor Hub Jumpers"
- note added: "ISM330DHCX MODES MODE1: Perhipheral-only mode I2C or SPI MODE2: Sensor Hub mode I2C or SPI with controller I2C port"
- note added: "If using Mode 2 (Sensor Hub Mode), cut both traces."
- note removed: "Accelerometer Address Selection Jumpers"
- moved on the sheet: 6DOF_ADDR, C1, C2, R5, R6, R7, U2
