File: Qwiic/SparkFun_9DoF_ISM330DHCX-MMC5983MA.sch (EAGLE design)
At the start: 35 parts, among them J1 QWIIC_RIGHT_ANGLE, J2 QWIIC_RIGHT_ANGLE, U1 ISM330DHCX, U2 MMC5983MA_QFN16

Commit message: Rolls to version v02
Other:
- note added: "v02"
- note removed: "v01"
Changed lines of the file:
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@@
 <text x="58.166" y="264.414" size="1.27" layer="97" font="vector">VDD Range: 1.71V - 3.6V
 VDDIO Range: 1.62V - 3.6V</text>
-<text x="421.64" y="7.62" size="2.54" layer="94" font="vector">v01</text>
+<text x="421.64" y="7.62" size="2.54" layer="94" font="vector">v02</text>
 <text x="170.18" y="68.58" size="1.778" layer="97" font="vector">Cut trace to
 disconnect Power

Commit message: Rolls to v10, adds silk to accelerometer address selection jumper
* Adds note to schematic about magnetometer address not being affected by accelerometer address selection
* Increases size of  VCC and address text
Other:
- note added: "Magnetometer address unaffected, no alternate address available."
- note added: "v10"
- note removed: "v02"
- moved on the sheet: U2
Changed lines of the file:
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@@
 <text x="216.916" y="103.632" size="1.778" layer="97" font="vector" align="top-left">Cut traces to remove I2C
 pull-up resistors.</text>
-<text x="58.166" y="264.414" size="1.27" layer="97" font="vector">VDD Range: 1.71V - 3.6V
+<text x="53.086" y="259.334" size="1.778" layer="97" font="vector">VDD Range: 1.71V - 3.6V
 VDDIO Range: 1.62V - 3.6V</text>
-<text x="421.64" y="7.62" size="2.54" layer="94" font="vector">v02</text>
+<text x="421.64" y="7.62" size="2.54" layer="94" font="vector">v10</text>
 <text x="170.18" y="68.58" size="1.778" layer="97" font="vector">Cut trace to
 disconnect Power
@@
 <wire x1="187.96" y1="228.6" x2="186.944" y2="227.838" width="0.2032" layer="97" style="dashdot"/>
 <text x="350.774" y="11.176" size="2.54" layer="94" font="vector">Elias Santistevan</text>
-<text x="315.722" y="257.556" size="1.27" layer="97" font="vector">VDD Range: 2.8V - 3.6V
+<text x="313.182" y="260.096" size="1.778" layer="97" font="vector">VDD Range: 2.8V - 3.6V
 VDDIO Range: 2.8V - 3.6V</text>
 <wire x1="0" y1="152.4" x2="137.16" y2="152.4" width="0.2032" layer="97" style="longdash"/>
@@
 Sensor Hub Jumpers</text>
 <text x="190.5" y="142.24" size="2.54" layer="94" font="vector" align="center">I2C and LED Jumpers</text>
-<text x="328.676" y="251.968" size="1.27" layer="97" font="vector" align="center">I2C address: 0x30</text>
+<text x="331.216" y="254.508" size="1.778" layer="97" font="vector" align="center">I2C address: 0x30</text>
 <text x="209.296" y="222.758" size="1.778" layer="97" font="vector">(Default)</text>
-<text x="50.8" y="259.08" size="1.27" layer="97" font="vector">I2C Address (selectable): 0x6B (Default)</text>
+<text x="43.18" y="254" size="1.778" layer="97" font="vector">I2C Address (selectable): 0x6B (Default)</text>
 <text x="48.26" y="182.88" size="1.778" layer="97" font="vector" align="top-left">ISM330DHCX MODES
 MODE1:  Perhipheral-only mode
@@
 <text x="208.28" y="162.306" size="1.778" layer="97" font="vector" rot="R180" align="top-left">If using Mode 2 (Sensor Hub Mode),
 cut both traces. </text>
+<text x="185.42" y="200.66" size="1.778" layer="97" font="vector">Magnetometer address unaffected,
+no alternate address available. </text>
 </plain>
 <instances>
@@
 <attribute name="REV" x="419.1" y="6.604" size="2.7432" layer="94" font="vector"/>
 </instance>
-<instance part="U2" gate="G$1" x="317.5" y="200.66" smashed="yes">
+<instance part="U2" gate="G$1" x="325.12" y="208.28" smashed="yes">
 <attribute name="NAME" x="317.5" y="217.17" size="1.778" layer="95"/>
-<attribute name="VALUE" x="317.5" y="198.12" size="1.778" layer="96"/>
+<attribute name="VALUE" x="314.96" y="198.12" size="1.778" layer="96"/>
 </instance>
 <instance part="SUPPLY7" gate="G$1" x="294.64" y="215.9" smashed="yes">
 <attribute name="VALUE" x="294.64" y="218.694" size="1.778" layer="96" align="bottom-center"/>
 </instance>
-<instance part="GND1" gate="1" x="312.42" y="193.04" smashed="yes">
-<attribute name="VALUE" x="312.42" y="192.786" size="1.778" layer="96" align="top-center"/>
+<instance part="GND1" gate="1" x="309.88" y="193.04" smashed="yes">
+<attribute name="VALUE" x="309.88" y="192.786" size="1.778" layer="96" align="top-center"/>
 </instance>
 <instance part="C1" gate="G$1" x="294.64" y="200.66" smashed="yes">
@@
 <segment>
 <pinref part="GND1" gate="1" pin="GND"/>
-<wire x1="312.42" y1="203.2" x2="312.42" y2="195.58" width="0.1524" layer="91"/>
+<wire x1="312.42" y1="203.2" x2="309.88" y2="203.2" width="0.1524" layer="91"/>
+<wire x1="309.88" y1="203.2" x2="309.88" y2="195.58" width="0.1524" layer="91"/>
 <pinref part="U2" gate="G$1" pin="GND"/>
-<wire x1="312.42" y1="203.2" x2="314.96" y2="203.2" width="0.1524" layer="91"/>
 </segment>
 <segment>
@@
 <wire x1="294.64" y1="215.9" x2="294.64" y2="213.36" width="0.1524" layer="91"/>
 <pinref part="U2" gate="G$1" pin="VDDIO"/>
-<wire x1="294.64" y1="213.36" x2="314.96" y2="213.36" width="0.1524" layer="91"/>
+<wire x1="294.64" y1="213.36" x2="312.42" y2="213.36" width="0.1524" layer="91"/>
 <pinref part="U2" gate="G$1" pin="VDD"/>
-<wire x1="314.96" y1="210.82" x2="294.64" y2="210.82" width="0.1524" layer="91"/>
+<wire x1="312.42" y1="210.82" x2="294.64" y2="210.82" width="0.1524" layer="91"/>
 <wire x1="294.64" y1="210.82" x2="294.64" y2="213.36" width="0.1524" layer="91"/>
 <junction x="294.64" y="213.36"/>
@@
 <pinref part="C2" gate="G$1" pin="1"/>
 <wire x1="302.26" y1="205.74" x2="302.26" y2="208.28" width="0.1524" layer="91"/>
-<wire x1="314.96" y1="208.28" x2="302.26" y2="208.28" width="0.1524" layer="91"/>
-</segment>
-</net>
+<wire x1="312.42" y1="208.28" x2="302.26" y2="208.28" width="0.1524" layer="91"/>
+</segment>
+</net>
